File: kicad/audua.kicad_pcb (KiCad board)
At the start: 2 copper layers, 0 parts

Commit message: Done?!
Parts:
- added BT1: BATTERY, SMTM2032, B.Cu at (94.2, 41.9)
- added C1: C, SM0402_c, F.Cu at (93.9, 56.5)
- added C10: 10uF, SM0603_Capa, F.Cu at (61.0, 51.8)
- added C2: C, SM0402_c, F.Cu at (94.0, 52.1)
- added C3: C, SM0402_c, F.Cu at (92.5, 43.1)
- added C4: C, SM0402_c, F.Cu at (66.3, 51.6)
- added C5: C, SM0402_c, F.Cu at (80.9, 33.4)
- added C6: C, SM0402_c, F.Cu at (68.1, 51.6)
- added C7: C, SM0402_c, F.Cu at (70.1, 51.6)
- added C8: 50uF, SM0603_Capa, F.Cu at (97.5, 54.4)
- added C9: 10uF, SM0603_Capa, F.Cu at (106.8, 46.6)
- added D1: LED, LED-0603, F.Cu at (64.0, 51.6)
- added GS1: GS3, GS3, F.Cu at (82.5, 45.5)
- added GS2: GS3, GS3, F.Cu at (82.5, 41.4)
- added GS3: GS3, GS3, F.Cu at (80.5, 41.4)
- added GS4: GS3, GS3, F.Cu at (80.5, 45.5)
- added L1: 2.2uH, SM0805, F.Cu at (81.5, 35.1)
- added MIC1: SPU0414HR5H-SB, SPU0414HR5H-SB, F.Cu at (94.6, 54.2)
- added P1: CONN_4, PIN_ARRAY_4x1, F.Cu at (104.9, 50.8)
- added P2: CONN_1, TP, F.Cu at (83.2, 32.3)
- added P3: CONN_1, TP, F.Cu at (83.2, 31.0)
- added P4: CONN_1, TP, F.Cu at (90.7, 33.5)
- added P5: CONN_1, TP, F.Cu at (92.1, 33.5)
- added P6: CONN_1, TP, F.Cu at (86.1, 39.1)
- added R1: R, SM0402_r, F.Cu at (97.0, 52.1)
- added R2: R, SM0402_r, F.Cu at (88.9, 38.1)
- added R3: 1000K, SM0402_r, F.Cu at (79.2, 37.8)
- added SW1: SPST, PTS525SM10, B.Cu at (107.6, 34.5)
- added U1: STM32L051-32QFN, QFN32, F.Cu at (86.9, 34.0)
- added U2: MICROSD, MicroSD, F.Cu at (101.9, 38.4)
- added U3: TPS62740, DSS12, F.Cu at (81.5, 37.3)
Routing:
- net GND: track 0.00 -> 98.9 mm, vias 0 -> 4
- net VDD: track 0.00 -> 64.1 mm, vias 0 -> 3
- net VCC: track 0.00 -> 19.0 mm, vias 0 -> 2
- net /VSEL1: track 0.00 -> 11.3 mm
- net /VSEL4: track 0.00 -> 10.5 mm
- net /VSEL3: track 0.00 -> 6.58 mm
- net /VSEL2: track 0.00 -> 6.57 mm
- net N-0000022: track 0.00 -> 6.20 mm
- net /SPI1_SCK: track 0.00 -> 5.94 mm
- net /SPI1_MISO: track 0.00 -> 5.23 mm
- net N-0000017: track 0.00 -> 3.22 mm
- net N-0000010: track 0.00 -> 1.80 mm
- net N-0000018: track 0.00 -> 1.62 mm
- net N-000003: track 0.00 -> 1.57 mm
- net N-0000012: track 0.00 -> 1.55 mm
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Other:
- net class Default: clearance 0.254 -> 0.1524; trace_width 0.254 -> 0.1524
- rule trace_clearance: 0.254 -> 0.1524
- rule trace_min: 0.254 -> 0.1524
